File: node/ESP32 Node/production/design/node.sch (EAGLE design)
At the start: 58 parts

Commit message: Added Navio2 libraries
Parts:
- added POWER_HEADER: 61300611121, Headers:61300611121
Connections:
- net 1V8: now also POWER_HEADER.2
- net 2V5: now also POWER_HEADER.3
- net 3V3: now also POWER_HEADER.4
- net 5V: now also POWER_HEADER.5
- net GND: now also ESP32-WROOM-32U.EXP, POWER_HEADER.1, POWER_HEADER.6
Other:
- moved on the sheet: 868MHZ_ANTENNA, C1, C13, C14, C15, C16, C17, C18, C19, C2, C20, C21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
